File: FMCtoEdgeLS(THRU)/FMCtoEdgeLS_R.brd (EAGLE design)
At the start: 94.6 x 114.3 mm, 120 parts, among them J1 ASP-134602-01

Commit message: Added files via upload
Routing:
- net GND: track 386.2 -> 389.0 mm, vias 137 -> 140
- net F31: track 51.3 -> 52.4 mm
- net H31: track 108.4 -> 109.0 mm
Changed lines of the file:
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@@
 <wire x1="45.72" y1="12.7" x2="45.085" y2="13.335" width="0.1524" layer="1"/>
 <wire x1="45.72" y1="10.16" x2="45.72" y2="12.7" width="0.1524" layer="1"/>
-<wire x1="70.485" y1="10.16" x2="45.72" y2="10.16" width="0.1524" layer="1"/>
+<wire x1="60.96" y1="10.16" x2="70.485" y2="10.16" width="0.1524" layer="1"/>
+<wire x1="57.15" y1="10.16" x2="45.72" y2="10.16" width="0.1524" layer="1"/>
 <wire x1="74.295" y1="13.97" x2="70.485" y2="10.16" width="0.1524" layer="1"/>
 <wire x1="90.17" y1="13.97" x2="74.295" y2="13.97" width="0.1524" layer="1"/>
 <wire x1="91.44" y1="15.24" x2="90.17" y2="13.97" width="0.1524" layer="1"/>
+<wire x1="57.15" y1="10.16" x2="57.2128" y2="10.2228" width="0.1524" layer="1"/>
+<wire x1="57.2128" y1="10.2228" x2="57.2128" y2="10.36943125" width="0.1524" layer="1"/>
+<wire x1="58.27336875" y1="11.43" x2="59.69" y2="11.43" width="0.1524" layer="1"/>
+<wire x1="59.69" y1="11.43" x2="60.96" y2="10.16" width="0.1524" layer="1"/>
+<wire x1="57.2128" y1="10.36943125" x2="58.27336875" y2="11.43" width="0.1524" layer="1"/>
 </signal>
 <signal name="G9">
@@
 <wire x1="46.99" y1="14.9225" x2="46.6725" y2="15.24" width="0.1524" layer="1"/>
 <wire x1="46.99" y1="11.43" x2="46.99" y2="14.9225" width="0.1524" layer="1"/>
-<wire x1="64.135" y1="11.43" x2="46.99" y2="11.43" width="0.1524" layer="1"/>
+<wire x1="60.96" y1="11.43" x2="64.135" y2="11.43" width="0.1524" layer="1"/>
+<wire x1="46.99" y1="11.43" x2="57.785" y2="11.43" width="0.1524" layer="1"/>
 <wire x1="72.39" y1="19.685" x2="64.135" y2="11.43" width="0.1524" layer="1"/>
 <wire x1="74.6125" y1="21.9075" x2="72.39" y2="19.685" width="0.1524" layer="16"/>
@@
 <via x="72.39" y="19.685" extent="1-16" drill="0.35"/>
 <via x="74.6125" y="73.66" extent="1-16" drill="0.35"/>
+<wire x1="57.785" y1="11.43" x2="58.42" y2="12.065" width="0.1524" layer="1"/>
+<wire x1="58.42" y1="12.065" x2="60.325" y2="12.065" width="0.1524" layer="1"/>
+<wire x1="60.325" y1="12.065" x2="60.96" y2="11.43" width="0.1524" layer="1"/>
 </signal>
 <signal name="J24">
@@
 <via x="70.485" y="71.12" extent="1-16" drill="0.35"/>
 <via x="61.595" y="20.955" extent="1-16" drill="0.35"/>
-<via x="58.42" y="8.89" extent="1-16" drill="0.35"/>
 <via x="55.245" y="31.115" extent="1-16" drill="0.35"/>
 <via x="55.245" y="32.385" extent="1-16" drill="0.35"/>
@@
 <via x="68.58" y="75.565" extent="1-16" drill="0.35"/>
 <via x="38.735" y="94.615" extent="1-16" drill="0.35"/>
-<via x="76.835" y="5.08" extent="1-16" drill="0.35"/>
 <via x="76.835" y="1.905" extent="1-16" drill="0.35"/>
 <via x="71.755" y="14.605" extent="1-16" drill="0.35"/>
 <via x="74.295" y="17.78" extent="1-16" drill="0.35"/>
-<via x="78.105" y="12.7" extent="1-16" drill="0.35"/>
+<via x="74.93" y="12.7" extent="1-16" drill="0.35"/>
 <via x="30.48" y="54.61" extent="1-16" drill="0.35"/>
 <via x="36.195" y="54.61" extent="1-16" drill="0.35"/>
@@
 <via x="33.655" y="50.165" extent="1-16" drill="0.35"/>
 <via x="34.29" y="48.26" extent="1-16" drill="0.35"/>
+<via x="76.835" y="5.08" extent="1-16" drill="0.35"/>
+<via x="78.105" y="17.78" extent="1-16" drill="0.35"/>
+<via x="5.715" y="22.225" extent="1-16" drill="0.35"/>
+<via x="5.715" y="34.925" extent="1-16" drill="0.35"/>
+<wire x1="55.245" y1="8.255" x2="55.88" y2="7.62" width="0.1524" layer="1"/>
+<wire x1="55.88" y1="7.62" x2="57.785" y2="7.62" width="0.1524" layer="1"/>
+<via x="62.865" y="6.985" extent="1-16" drill="0.35"/>
 </signal>
 <signal name="K11">
@@
 <contactref element="U$1" pad="P$60"/>
 <wire x1="35.56" y1="8.89" x2="34.925" y2="9.525" width="0.1524" layer="1"/>
-<wire x1="35.56" y1="6.35" x2="35.56" y2="8.89" width="0.1524" layer="1"/>
-<wire x1="57.15" y1="6.35" x2="35.56" y2="6.35" width="0.1524" layer="1"/>
-<wire x1="60.6425" y1="9.8425" x2="57.15" y2="6.35" width="0.1524" layer="1"/>
-<wire x1="70.8025" y1="9.8425" x2="60.6425" y2="9.8425" width="0.1524" layer="1"/>
+<wire x1="35.56" y1="8.89" x2="35.56" y2="6.35" width="0.1524" layer="1"/>
+<wire x1="60.96" y1="6.35" x2="64.4525" y2="9.8425" width="0.1524" layer="1"/>
+<wire x1="70.8025" y1="9.8425" x2="64.4525" y2="9.8425" width="0.1524" layer="1"/>
 <wire x1="72.7075" y1="11.7475" x2="70.8025" y2="9.8425" width="0.1524" layer="1"/>
 <wire x1="80.645" y1="11.7475" x2="72.7075" y2="11.7475" width="0.1524" layer="1"/>
@@
 <via x="80.9625" y="12.065" extent="1-16" drill="0.35"/>
 <via x="82.55" y="73.66" extent="1-16" drill="0.35"/>
+<wire x1="57.24435" y1="6.35" x2="57.53365" y2="6.6393" width="0.1524" layer="1"/>
+<wire x1="57.53365" y1="6.6393" x2="58.03635" y2="6.6393" width="0.1524" layer="1"/>
+<wire x1="58.03635" y1="6.6393" x2="58.32565" y2="6.35" width="0.1524" layer="1"/>
+<wire x1="35.56" y1="6.35" x2="57.24435" y2="6.35" width="0.1524" layer="1"/>
+<wire x1="58.32565" y1="6.35" x2="60.96" y2="6.35" width="0.1524" layer="1"/>
 </signal>
 <signal name="C27">
